File: V1.0/PCB_Files/RTC_Module.kicad_pcb (KiCad board)
At the start: 2 copper layers, 42.1 x 18.5 mm, 17 parts, among them J1 DZ254W-11-06-65, U2 PCF8563T, U3 XC6206P332MR-G, Y1 Q13FC13500004

Commit message: This is ordered Version!!!
Parts:
- moved G*** 2.76 mm to (119.0, 75.7)
- moved BT1 1.33 mm to (128.7, 67.7)
Other:
- board size 42.1 x 18.5 mm -> 44.9 x 18.5 mm
Changed lines of the file:
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@@
 	(footprint "LOGO"
 		(layer "F.Cu")
-		(at 121.75323 75.5)
+		(at 119 75.7)
 		(property "Reference" "G***"
-			(at 0 0 360)
+			(at 0 0 0)
 			(layer "F.SilkS")
 			(hide yes)
@@
 		)
 		(property "Value" "LOGO"
-			(at 0.75 0 360)
+			(at 0.75 0 0)
 			(layer "F.SilkS")
 			(hide yes)
@@
 	)
 	(footprint "Battery:BatteryHolder_LINX_BAT-HLD-012-SMT"
-		(locked yes)
 		(layer "F.Cu")
-		(at 129.999999 67.6)
+		(at 128.675 67.675)
 		(descr "SMT battery holder for CR1216/1220/1225, https://linxtechnologies.com/wp/wp-content/uploads/bat-hld-012-smt.pdf")
 		(tags "battery holder coin cell cr1216 cr1220 cr1225")
 		(property "Reference" "BT1"
-			(at 7.900001 3.7 360)
+			(at 7.900001 3.7 0)
 			(layer "F.SilkS")
 			(effects
@@
 		)
 		(property "Value" "MY-1220-03"
-			(at 0 -6.999999 360)
+			(at 0 -6.999999 0)
 			(layer "F.Fab")
 			(effects
@@
 		)
 		(fp_text user "${REFERENCE}"
-			(at 0 0 360)
+			(at 0 0 0)
 			(layer "F.Fab")
 			(effects
@@
 		)
 		(pad "1" smd rect
-			(at -7.600001 0)
-			(size 2.5 5.1)
+			(at -8.325 0)
+			(size 3.949999 5.1)
 			(layers "F.Cu" "F.Paste" "F.Mask")
 			(net 2 "3.3V")
@@
 		)
 		(pad "1" smd rect
-			(at 7.600001 0)
-			(size 2.5 5.1)
+			(at 8.325 0.025)
+			(size 3.949999 5.05)
 			(layers "F.Cu" "F.Paste" "F.Mask")
 			(net 2 "3.3V")
@@
 		)
 		(property "Value" "1uF/10V"
-			(at 0 1.679999 270)
+			(at 0 1.679999 -90)
 			(layer "F.Fab")
 			(effects
@@
 		)
 		(fp_text user "${REFERENCE}"
-			(at 0 0 270)
+			(at 0 0 -90)
 			(layer "F.Fab")
 			(effects
@@
 		)
 		(property "Value" "XC6206P332MR-G"
-			(at 0 2.4 360)
+			(at 0 2.4 0)
 			(layer "F.Fab")
 			(effects
@@
 		)
 		(fp_text user "${REFERENCE}"
-			(at 0 0 360)
+			(at 0 0 0)
 			(layer "F.Fab")
 			(effects
@@
 	(gr_line
 		(start 162.1 77.7)
-		(end 120 77.7)
+		(end 117.2 77.7)
 		(stroke
 			(width 0.05)
@@
 	)
 	(gr_line
-		(start 120 77.7)
-		(end 120 59.2)
+		(start 117.2 77.7)
+		(end 117.2 59.2)
 		(stroke
 			(width 0.05)
@@
 	)
 	(gr_line
-		(start 120 59.2)
+		(start 117.2 59.2)
 		(end 162.1 59.2)
 		(stroke
@@
 	)
 	(gr_text "RTC Module V1.0"
-		(at 123.05323 76.5 0)
+		(at 120.3 76.7 0)
 		(layer "F.SilkS" knockout)
 		(effects
@@
 	)
 	(via
-		(at 138.3 61.4)
+		(at 121 62.2)
 		(size 0.6)
 		(drill 0.3)
@@
 	)
 	(via
-		(at 154.9 73.6)
+		(at 138.3 61.4)
 		(size 0.6)
 		(drill 0.3)
@@
 	)
 	(via
-		(at 147.6 65.9)
+		(at 154.9 73.6)
 		(size 0.6)
 		(drill 0.3)
@@
 	)
 	(via
-		(at 135.4 65.1)
+		(at 147.6 65.9)
 		(size 0.6)
 		(drill 0.3)
@@
 	)
 	(via
-		(at 124.7 70.3)
+		(at 139.6 63.9)
 		(size 0.6)
 		(drill 0.3)
@@
 	)
 	(via
-		(at 139.6 63.9)
+		(at 130.2 73.6)
 		(size 0.6)
 		(drill 0.3)
@@
 	)
 	(via
-		(at 135.2 76.1)
+		(at 132.5 76.3)
 		(size 0.6)
 		(drill 0.3)
@@
 	)
 	(via
-		(at 124.9 64.3)
+		(at 147.7 67.2)
 		(size 0.6)
 		(drill 0.3)
@@
 	)
 	(via
-		(at 147.7 67.2)
+		(at 147.9 62.7)
 		(size 0.6)
 		(drill 0.3)
@@
 	)
 	(via
-		(at 147.9 62.7)
+		(at 136.4 73.5)
 		(size 0.6)
 		(drill 0.3)
@@
 	)
 	(via
-		(at 135.4 70.4)
+		(at 121.6 73.3)
 		(size 0.6)
 		(drill 0.3)
@@
 	)
 	(segment
+		(start 144.37 70.400001)
+		(end 143.269999 69.3)
+		(width 0.5)
+		(layer "F.Cu")
+		(net 2)
+	)
+	(segment
 		(start 150.9625 70.649999)
 		(end 152.025 71.712499)
@@
 	)
 	(segment
-		(start 143.069999 69.1)
-		(end 139.1 69.1)
-		(width 0.5)
-		(layer "F.Cu")
-		(net 2)
-	)
-	(segment
-		(start 148.8 70.649999)
-		(end 150.9625 70.649999)
-		(width 0.5)
-		(layer "F.Cu")
-		(net 2)
-	)
-	(segment
-		(start 137.6 65)
-		(end 133.9 61.3)
+		(start 138.6 69.3)
+		(end 137 67.7)
 		(width 0.5)
 		(layer "F.Cu")
@@
 	)
 	(segment
-		(start 138.4 69.4)
-		(end 137.5 68.5)
+		(start 132.8 61.4)
+		(end 124 61.4)
 		(width 0.5)
 		(layer "F.Cu")
@@
 	)
 	(segment
-		(start 137.6 67.6)
-		(end 137.6 65)
+		(start 148.8 70.649999)
+		(end 150.9625 70.649999)
 		(width 0.5)
 		(layer "F.Cu")
@@
 	)
 	(segment
-		(start 122.399998 65.000002)
-		(end 122.399998 67.6)
+		(start 143.269999 69.3)
+		(end 138.6 69.3)
 		(width 0.5)
 		(layer "F.Cu")
@@
 	)
 	(segment
-		(start 133.9 61.3)
-		(end 126.1 61.3)
-		(width 0.5)
-		(layer "F.Cu")
-		(net 2)
-	)
-	(segment
 		(start 146.065 71.875)
 		(end 146.825 72.635)
@@
 	)
 	(segment
-		(start 126.1 61.3)
-		(end 122.399998 65.000002)
+		(start 120.35 65.05)
+		(end 120.35 67.675)
 		(width 0.5)
 		(layer "F.Cu")
@@
 	)
 	(segment
-		(start 139.1 69.1)
-		(end 137.6 67.6)
+		(start 137 65.6)
+		(end 132.8 61.4)
 		(width 0.5)
 		(layer "F.Cu")
@@
 	)
 	(segment
+		(start 124 61.4)
+		(end 120.35 65.05)
+		(width 0.5)
+		(layer "F.Cu")
+		(net 2)
+	)
+	(segment
+		(start 137 67.7)
+		(end 137 65.6)
+		(width 0.5)
+		(layer "F.Cu")
+		(net 2)
+	)
+	(segment
 		(start 146.065 71.875)
 		(end 144.87 71.875)
@@
 	)
 	(segment
-		(start 144.37 70.400001)
-		(end 143.069999 69.1)
-		(width 0.5)
-		(layer "F.Cu")
-		(net 2)
-	)
-	(segment
 		(start 152.175 64.6)
 		(end 153.45 64.6)
@@
 		(polygon
 			(pts
-				(xy 117.5 56.5) (xy 163.5 56.5) (xy 163.5 80) (xy 117.5 80)
+				(xy 115 56.5) (xy 163.5 56.5) (xy 163.5 80) (xy 115 80)
 			)
 		)
